File: msp-7seg.sch (KiCad schematic (older format))
At the start: 30 parts, among them P1 CONN_11, P3 I2C, Q1 PNP, Q2 PNP, Q3 PNP, Q4 PNP, U1 MSP430G2553IN20, U2 74HC595, U3 LP2985LV, X1 CRYSTAL

Commit message: Spread out components and added reset button
Parts:
- added C5: 1nF, symbol C
- added SW1: RESET, symbol SW_PUSH
- U1: value MSP430G2553IN20 -> MSP430G2553
- U3: value LP2985LV -> 2985
Connections:
- net A: now also R6.1; no longer R3.1
- net C: now also R7.1; no longer R2.1
- net D: now also R3.1; no longer R7.1
- net DP: now also R1.1; no longer R8.1
- net E: now also R2.1; no longer R6.1
- net F: now also R8.1; no longer R1.1
- net GND: now also C5.2, SW1.1
- net RESET: now also C5.1, SW1.2
Changed lines of the file:
@@
 P 3100 5600
 F 0 "U1" H 3100 4800 60  0000 C CNN
-F 1 "MSP430G2553IN20" H 3100 6450 60  0000 C CNN
+F 1 "MSP430G2553" H 3100 6450 60  0000 C CNN
 F 2 "" H 3100 5600 60  0000 C CNN
 F 3 "" H 3100 5600 60  0000 C CNN
@@
 	0    -1   -1   0
 $EndComp
-Wire Wire Line
-	9550 1250 9550 1400
-Wire Wire Line
-	9550 2650 9550 2500
-Wire Wire Line
-	10200 1500 9950 1500
-Wire Wire Line
-	2200 5050 2400 5050
-Wire Wire Line
-	10200 1700 9950 1700
-Wire Wire Line
-	10200 2000 9950 2000
-Wire Wire Line
-	10050 2150 10050 2100
-Wire Wire Line
-	10050 2100 9950 2100
-Wire Wire Line
-	10150 1800 9950 1800
-Wire Wire Line
-	4050 2950 4050 2900
-Wire Wire Line
-	4950 2900 4950 2950
-Wire Wire Line
-	4650 2900 4650 2950
-Wire Wire Line
-	4350 2900 4350 2950
 Text Label 4000 1500 1    60   ~ 0
 B
@@
 Text Label 8050 1800 2    60   ~ 0
 B
+Text Label 8050 1700 2    60   ~ 0
+D
+Text Label 8050 1600 2    60   ~ 0
+E
+Text Label 8050 1500 2    60   ~ 0
+DP
 Text Label 8050 2100 2    60   ~ 0
-D
+C
 Text Label 8050 2000 2    60   ~ 0
-E
+A
 Text Label 8050 2200 2    60   ~ 0
-DP
-Text Label 8050 1600 2    60   ~ 0
-C
-Text Label 8050 1700 2    60   ~ 0
-A
-Text Label 8050 1500 2    60   ~ 0
 F
 $Comp
@@
 	1    0    0    -1
 $EndComp
-Wire Wire Line
-	1900 5750 1900 5800
 $Comp
 L VCC #PWR06
@@
 	1    0    0    -1
 $EndComp
-Wire Wire Line
-	2350 4350 2350 4900
-Wire Wire Line
-	2350 4900 2400 4900
 $Comp
 L GND #PWR010
@@
 	1    0    0    -1
 $EndComp
-Wire Wire Line
-	3900 4950 3900 4900
-Wire Wire Line
-	3900 4900 3800 4900
 Text Label 4000 5050 0    60   ~ 0
 XIN
 Text Label 4000 5200 0    60   ~ 0
 XOUT
-Wire Wire Line
-	4000 5200 3800 5200
-Wire Wire Line
-	4000 5050 3800 5050
 Text Label 4000 5350 0    60   ~ 0
 TEST
 Text Label 4000 5500 0    60   ~ 0
 RESET
-Wire Wire Line
-	4000 5350 3800 5350
-Wire Wire Line
-	4000 5500 3800 5500
 Text Label 4000 5650 0    60   ~ 0
 P1.7
 Text Label 4000 5800 0    60   ~ 0
 P1.6
-Wire Wire Line
-	4000 5650 3800 5650
-Wire Wire Line
-	4000 5800 3800 5800
 Text Label 2400 5200 2    60   ~ 0
 P1.1
@@
 P 6000 4000
 F 0 "U3" H 6200 3550 60  0000 C CNN
-F 1 "LP2985LV" H 6000 4450 60  0000 C CNN
+F 1 "2985" H 6000 4450 60  0000 C CNN
 F 2 "" H 6000 4000 60  0000 C CNN
 F 3 "" H 6000 4000 60  0000 C CNN
@@
 	1    0    0    -1
 $EndComp
-Wire Wire Line
-	5200 4200 5100 4200
 $Comp
 L GND #PWR011
@@
 	1    0    0    -1
 $EndComp
-Wire Wire Line
-	6000 4700 6000 4750
-Wire Wire Line
-	4900 4700 6950 4700
-Wire Wire Line
-	5100 4700 5100 4600
 $Comp
 L C C1
@@
 	1    0    0    -1
 $EndComp
-Wire Wire Line
-	4900 4100 4900 4700
-Connection ~ 5100 4700
-Wire Wire Line
-	5200 3700 5200 3900
 $Comp
 L C C3
@@
 	0    1    1    0
 $EndComp
-Wire Wire Line
-	6800 3700 7150 3700
-Connection ~ 6950 3700
-Wire Wire Line
-	6950 4700 6950 4100
-Connection ~ 6000 4700
 $Comp
 L R R9
@@
 	0    -1   -1   0
 $EndComp
-Wire Wire Line
-	1750 6100 1700 6100
-Wire Wire Line
-	1750 6250 1250 6250
 $Comp
 L R R12
@@
 	0    -1   -1   0
 $EndComp
-Wire Wire Line
-	3950 5950 3800 5950
-Wire Wire Line
-	3950 6100 3800 6100
-Wire Wire Line
-	4600 5950 4450 5950
-Wire Wire Line
-	4450 6100 5250 6100
-Wire Wire Line
-	2250 6250 2400 6250
-Wire Wire Line
-	2400 6100 2250 6100
 Text Label 8550 3750 2    60   ~ 0
 Vin
@@
 	1    0    0    -1
 $EndComp
-Wire Wire Line
-	8350 3850 8350 4000
-Wire Wire Line
-	8350 3950 8550 3950
 Text Label 8550 4150 2    60   ~ 0
 P1.1
@@
 Text Label 8550 4650 2    60   ~ 0
 P1.7
-Wire Wire Line
-	8550 3850 8350 3850
-Connection ~ 8350 3950
 $Comp
 L CONN_4 P3
@@
 	1    0    0    -1
 $EndComp
-Wire Wire Line
-	9900 3300 9700 3300
-Wire Wire Line
-	9700 3300 9700 3200
 Text Label 3800 5650 0    60   ~ 0
 SDA
@@
 	0    1    1    0
 $EndComp
-Wire Wire Line
-	3150 2300 3050 2300
 $Comp
 L R R14
@@
 	0    -1   -1   0
 $EndComp
-Wire Wire Line
-	5900 2100 5850 2100
 $Comp
 L GND #PWR017
@@
 	1    0    0    -1
 $EndComp
-Wire Wire Line
-	6500 2400 6500 2100
-Wire Wire Line
-	6500 2100 6400 2100
 $Comp
 L VCC #PWR018
@@
 	1    0    0    -1
 $EndComp
-Wire Wire Line
-	6300 5100 6300 5150
 $Comp
 L C C4
@@
 $EndComp
 $Comp
-L GND #PWR020
+L GND #PWR019
 U 1 1 5304EB32
 P 2100 4900
-F 0 "#PWR020" H 2100 4900 30  0001 C CNN
+F 0 "#PWR019" H 2100 4900 30  0001 C CNN
 F 1 "GND" H 2100 4830 30  0001 C CNN
 F 2 "" H 2100 4900 60  0000 C CNN
@@
 	1    0    0    -1
 $EndComp
-Wire Wire Line
-	2100 4900 2100 4850
-Wire Wire Line
-	2100 4450 2350 4450
-Connection ~ 2350 4450
 Text Label 2550 2300 2    60   ~ 0
 P1.3
@@
 Text Notes 6050 2500 0    60   ~ 0
 DNP
-Wire Wire Line
-	4650 3700 5200 3700
-Connection ~ 4900 3700
 $Comp
 L CONN_11 P1
@@
 	1    0    0    -1
 $EndComp
-Wire Wire Line
-	9800 3650 9800 3600
-Wire Wire Line
-	9800 3600 9900 3600
 Text Label 6500 5750 0    60   ~ 0
 RESET
-Wire Wire Line
-	6300 5750 6500 5750
-Wire Wire Line
-	6300 5650 6300 5750
+$Comp
+L GND #PWR020
+U 1 1 5304E784
+P 6300 6300
+F 0 "#PWR020" H 6300 6300 30  0001 C CNN
+F 1 "GND" H 6300 6230 30  0001 C CNN
+F 2 "" H 6300 6300 60  0000 C CNN
+F 3 "" H 6300 6300 60  0000 C CNN
+	1    6300 6300
+	1    0    0    -1
+$EndComp
+$Comp
+L C C5
+U 1 1 5304E7AC
+P 6300 6050
+F 0 "C5" H 6300 6150 40  0000 L CNN
+F 1 "1nF" H 6306 5965 40  0000 L CNN
+F 2 "" H 6338 5900 30  0000 C CNN
+F 3 "" H 6300 6050 60  0000 C CNN
+	1    6300 6050
+	1    0    0    -1
+$EndComp
+Wire Wire Line
+	9550 1250 9550 1400
+Wire Wire Line
+	9550 2650 9550 2500
+Wire Wire Line
+	10200 1500 9950 1500
+Wire Wire Line
+	2200 5050 2400 5050
+Wire Wire Line
+	10200 1700 9950 1700
+Wire Wire Line
+	10200 2000 9950 2000
+Wire Wire Line
+	10050 2150 10050 2100
+Wire Wire Line
+	10050 2100 9950 2100
+Wire Wire Line
+	10150 1800 9950 1800
+Wire Wire Line
+	4050 2950 4050 2900
+Wire Wire Line
+	4950 2900 4950 2950
+Wire Wire Line
+	4650 2900 4650 2950
+Wire Wire Line
+	4350 2900 4350 2950
+Wire Wire Line
+	1900 5750 1900 5800
+Wire Wire Line
+	2350 4350 2350 4900
+Wire Wire Line
+	2350 4900 2400 4900
+Wire Wire Line
+	3900 4950 3900 4900
+Wire Wire Line
+	3900 4900 3800 4900
+Wire Wire Line
+	4000 5200 3800 5200
+Wire Wire Line
+	4000 5050 3800 5050
+Wire Wire Line
+	4000 5350 3800 5350
+Wire Wire Line
+	4000 5500 3800 5500
+Wire Wire Line
+	4000 5650 3800 5650
+Wire Wire Line
+	4000 5800 3800 5800
+Wire Wire Line
+	5200 4200 5100 4200
+Wire Wire Line
+	6000 4700 6000 4750
+Wire Wire Line
+	4900 4700 6950 4700
+Wire Wire Line
+	5100 4700 5100 4600
+Wire Wire Line
+	4900 4100 4900 4700
+Connection ~ 5100 4700
+Wire Wire Line
+	5200 3700 5200 3900
+Wire Wire Line
+	6800 3700 7150 3700
+Connection ~ 6950 3700
+Wire Wire Line
+	6950 4700 6950 4100
+Connection ~ 6000 4700
+Wire Wire Line
+	1750 6100 1700 6100
+Wire Wire Line
+	1750 6250 1250 6250
+Wire Wire Line
+	3950 5950 3800 5950
+Wire Wire Line
+	3950 6100 3800 6100
+Wire Wire Line
+	4600 5950 4450 5950
+Wire Wire Line
+	4450 6100 5250 6100
+Wire Wire Line
+	2250 6250 2400 6250
+Wire Wire Line
+	2400 6100 2250 6100
+Wire Wire Line
+	8350 3850 8350 4000
+Wire Wire Line
+	8350 3950 8550 3950
+Wire Wire Line
+	8550 3850 8350 3850
+Connection ~ 8350 3950
+Wire Wire Line
+	9900 3300 9700 3300
+Wire Wire Line
+	9700 3300 9700 3200
+Wire Wire Line
+	3150 2300 3050 2300
+Wire Wire Line
+	5900 2100 5850 2100
+Wire Wire Line
+	6500 2400 6500 2100
+Wire Wire Line
+	6500 2100 6400 2100
+Wire Wire Line
+	6300 5100 6300 5150
+Wire Wire Line
+	6300 5650 6300 5850
+Connection ~ 6300 5750
+Wire Wire Line
+	6300 6250 6300 6300
+Wire Wire Line
+	2100 4900 2100 4850
+Wire Wire Line
+	2100 4450 2350 4450
+Connection ~ 2350 4450
+Wire Wire Line
+	4650 3700 5200 3700
+Connection ~ 4900 3700
+Wire Wire Line
+	9800 3650 9800 3600
+Wire Wire Line
+	9800 3600 9900 3600
+Wire Wire Line
+	6250 5750 6500 5750
+$Comp
+L GND #PWR021
+U 1 1 530E3F6C
+P 5650 5850
+F 0 "#PWR021" H 5650 5850 30  0001 C CNN
+F 1 "GND" H 5650 5780 30  0001 C CNN
+F 2 "" H 5650 5850 60  0000 C CNN
+F 3 "" H 5650 5850 60  0000 C CNN
+	1    5650 5850
+	1    0    0    -1
+$EndComp
+Wire Wire Line
+	5650 5850 5650 5750
+$Comp
+L SW_PUSH SW1
+U 1 1 530E48AE
+P 5950 5750
+F 0 "SW1" H 6100 5860 50  0000 C CNN
+F 1 "RESET" H 5950 5670 50  0000 C CNN
+F 2 "" H 5950 5750 60  0000 C CNN
+F 3 "" H 5950 5750 60  0000 C CNN
+	1    5950 5750
+	1    0    0    -1
+$EndComp
 $EndSCHEMATC

Commit message: Cleaned up silkscreen, added gerbers, schematic and images
Parts:
- X1: value CRYSTAL -> 32KHz
Changed lines of the file:
@@
 encoding utf-8
 Sheet 1 1
-Title ""
-Date ""
+Title "Mini Sapphire Prototyping 7segment"
+Date "26 feb 2014"
 Rev ""
-Comp ""
-Comment1 ""
+Comp "Niels Kjøller Hansen"
+Comment1 "Licensed under CERN OHL v.1.2"
 Comment2 ""
 Comment3 ""
@@
 P 9550 5950
 F 0 "X1" H 9550 6100 60  0000 C CNN
-F 1 "CRYSTAL" H 9550 5800 60  0000 C CNN
+F 1 "32KHz" H 9550 5800 60  0000 C CNN
 F 2 "" H 9550 5950 60  0000 C CNN
 F 3 "" H 9550 5950 60  0000 C CNN

Commit message: Added breakout for shift register
Parts:
- added P2: Serial, symbol CONN_5
- P1: value CONN_11 -> IO
Connections:
- net GND: now also P2.5
- net SerialClock: now also P2.3
- net SerialLatch: now also P2.4
- net VCC: now also P2.1
- net SerialOut: now reaches U2.9 (~QH)
- net SerialOut: now also P2.2
Other:
- moved on the sheet: P3, X1
Changed lines of the file:
@@
 L CRYSTAL X1
 U 1 1 52FF84C1
-P 9550 5950
-F 0 "X1" H 9550 6100 60  0000 C CNN
-F 1 "32KHz" H 9550 5800 60  0000 C CNN
-F 2 "" H 9550 5950 60  0000 C CNN
-F 3 "" H 9550 5950 60  0000 C CNN
-	1    9550 5950
-	1    0    0    -1
-$EndComp
-Text Label 9250 5950 2    60   ~ 0
+P 2700 7000
+F 0 "X1" H 2700 7150 60  0000 C CNN
+F 1 "32KHz" H 2700 6850 60  0000 C CNN
+F 2 "" H 2700 7000 60  0000 C CNN
+F 3 "" H 2700 7000 60  0000 C CNN
+	1    2700 7000
+	1    0    0    -1
+$EndComp
+Text Label 2400 7000 2    60   ~ 0
 XIN
-Text Label 9850 5950 0    60   ~ 0
+Text Label 3000 7000 0    60   ~ 0
 XOUT
 $Comp
@@
 L CONN_4 P3
 U 1 1 5303C34F
-P 10250 3450
-F 0 "P3" V 10200 3450 50  0000 C CNN
-F 1 "I2C" V 10300 3450 50  0000 C CNN
-F 2 "" H 10250 3450 60  0000 C CNN
-F 3 "" H 10250 3450 60  0000 C CNN
-	1    10250 3450
+P 10150 4500
+F 0 "P3" V 10100 4500 50  0000 C CNN
+F 1 "I2C" V 10200 4500 50  0000 C CNN
+F 2 "" H 10150 4500 60  0000 C CNN
+F 3 "" H 10150 4500 60  0000 C CNN
+	1    10150 4500
 	1    0    0    -1
 $EndComp
@@
 L VCC #PWR015
 U 1 1 5303C376
-P 9700 3200
-F 0 "#PWR015" H 9700 3300 30  0001 C CNN
-F 1 "VCC" H 9700 3300 30  0000 C CNN
-F 2 "" H 9700 3200 60  0000 C CNN
-F 3 "" H 9700 3200 60  0000 C CNN
-	1    9700 3200
+P 9600 4250
+F 0 "#PWR015" H 9600 4350 30  0001 C CNN
+F 1 "VCC" H 9600 4350 30  0000 C CNN
+F 2 "" H 9600 4250 60  0000 C CNN
+F 3 "" H 9600 4250 60  0000 C CNN
+	1    9600 4250
 	1    0    0    -1
 $EndComp
@@
 L GND #PWR016
 U 1 1 5303C38A
-P 9800 3650
-F 0 "#PWR016" H 9800 3650 30  0001 C CNN
-F 1 "GND" H 9800 3580 30  0001 C CNN
-F 2 "" H 9800 3650 60  0000 C CNN
-F 3 "" H 9800 3650 60  0000 C CNN
-	1    9800 3650
+P 9700 4700
+F 0 "#PWR016" H 9700 4700 30  0001 C CNN
+F 1 "GND" H 9700 4630 30  0001 C CNN
+F 2 "" H 9700 4700 60  0000 C CNN
+F 3 "" H 9700 4700 60  0000 C CNN
+	1    9700 4700
 	1    0    0    -1
 $EndComp
@@
 Text Label 3800 5800 0    60   ~ 0
 SCL
-Text Label 9900 3500 2    60   ~ 0
+Text Label 9800 4550 2    60   ~ 0
 TEST
-Text Label 9900 3400 2    60   ~ 0
+Text Label 9800 4450 2    60   ~ 0
 RESET
 $Comp
@@
 P 8900 4250
 F 0 "P1" V 8850 4250 60  0000 C CNN
-F 1 "CONN_11" V 8950 4250 60  0000 C CNN
+F 1 "IO" V 8950 4250 60  0000 C CNN
 F 2 "" H 8900 4250 60  0000 C CNN
 F 3 "" H 8900 4250 60  0000 C CNN
@@
 Connection ~ 8350 3950
 Wire Wire Line
-	9900 3300 9700 3300
-Wire Wire Line
-	9700 3300 9700 3200
+	9800 4350 9600 4350
+Wire Wire Line
+	9600 4350 9600 4250
 Wire Wire Line
 	3150 2300 3050 2300
@@
 Connection ~ 4900 3700
 Wire Wire Line
-	9800 3650 9800 3600
-Wire Wire Line
-	9800 3600 9900 3600
+	9700 4700 9700 4650
+Wire Wire Line
+	9700 4650 9800 4650
 Wire Wire Line
 	6250 5750 6500 5750
@@
 	1    0    0    -1
 $EndComp
+Text Label 8400 2400 2    60   ~ 0
+SerialOut
+Wire Wire Line
+	8550 2400 8400 2400
+$Comp
+L CONN_5 P2
+U 1 1 5311A400
+P 10200 3300
+F 0 "P2" V 10150 3300 50  0000 C CNN
+F 1 "Serial" V 10250 3300 50  0000 C CNN
+F 2 "" H 10200 3300 60  0000 C CNN
+F 3 "" H 10200 3300 60  0000 C CNN
+	1    10200 3300
+	1    0    0    -1
+$EndComp
+$Comp
+L VCC #PWR022
+U 1 1 5311A45D
+P 9700 3000
+F 0 "#PWR022" H 9700 3100 30  0001 C CNN
+F 1 "VCC" H 9700 3100 30  0000 C CNN
+F 2 "" H 9700 3000 60  0000 C CNN
+F 3 "" H 9700 3000 60  0000 C CNN
+	1    9700 3000
+	1    0    0    -1
+$EndComp
+$Comp
+L GND #PWR023
+U 1 1 5311A471
+P 9700 3650
+F 0 "#PWR023" H 9700 3650 30  0001 C CNN
+F 1 "GND" H 9700 3580 30  0001 C CNN
+F 2 "" H 9700 3650 60  0000 C CNN
+F 3 "" H 9700 3650 60  0000 C CNN
+	1    9700 3650
+	1    0    0    -1
+$EndComp
+Wire Wire Line
+	9700 3650 9700 3500
+Wire Wire Line
+	9700 3500 9800 3500
+Wire Wire Line
+	9700 3000 9700 3100
+Wire Wire Line
+	9700 3100 9800 3100
+Text Label 9750 3200 2    60   ~ 0
+SerialOut
+Text Label 9750 3300 2    60   ~ 0
+SerialClock
+Text Label 9750 3400 2    60   ~ 0
+SerialLatch
+Wire Wire Line
+	9800 3200 9750 3200
+Wire Wire Line
+	9800 3300 9750 3300
+Wire Wire Line
+	9800 3400 9750 3400
 $EndSCHEMATC
